Commit message: fix: repeated link names

File: custom_dual_ee_description/urdf/end-effector-left.urdf.xacro (robot description, xacro)
@@ -17,5 +17,5 @@
   <xacro:macro name="end_effector_left" params="parent *origin">
     <!-- Example link and Joint -->
-    <link name="cee_tool_link">
+    <link name="cee_left_tool_link">
       <inertial>
         <origin xyz="0 0 0" rpy="0 0 0" />
@@ -41,8 +41,8 @@
       </collision>
     </link>
-    <joint name="cee_tool_joint" type="fixed">
+    <joint name="cee_left_tool_joint" type="fixed">
       <xacro:insert_block name="origin"/>
       <parent link="${parent}" />
-      <child link="cee_tool_link" />
+      <child link="cee_left_tool_link" />
       <axis xyz="0 0 0" />
     </joint>

File: custom_dual_ee_description/urdf/end-effector-right.urdf.xacro (robot description, xacro)
@@ -17,5 +17,5 @@
   <xacro:macro name="end_effector_right" params="parent *origin">
     <!-- Example link and Joint -->
-    <link name="cee_tool_link">
+    <link name="cee_right_tool_link">
       <inertial>
         <origin xyz="0 0 0" rpy="0 0 0" />
@@ -41,8 +41,8 @@
       </collision>
     </link>
-    <joint name="cee_tool_joint" type="fixed">
+    <joint name="cee_right_tool_joint" type="fixed">
       <xacro:insert_block name="origin"/>
       <parent link="${parent}" />
-      <child link="cee_tool_link" />
+      <child link="cee_right_tool_link" />
       <axis xyz="0 0 0" />
     </joint>
